File: hardware/KiCad/3_Connectors.kicad_sch (KiCad schematic)
At the start: 20 parts

Commit message: updates
Parts:
- removed BOOT1: BOOT, ProPrj_STM-easyedapro:HDR-F-2.54_1X3, symbol ProPrj_STM-easyedapro:BOOT
- removed C25: 100nF, ProPrj_STM-easyedapro:C0603, symbol ProPrj_STM-easyedapro:100nF
- removed GPIO1: HDR-F-2.54_1x8, ProPrj_STM-easyedapro:HDR-F-2.54_1X8, symbol ProPrj_STM-easyedapro:HDR-F-2.54_1x8
- removed I2C1: I2C, ProPrj_STM-easyedapro:JST-XH-04-PACKAGE-LONG-PAD, symbol ProPrj_STM-easyedapro:I2C
- removed R30, R31: 10kΩ, ProPrj_STM-easyedapro:R0402, symbol ProPrj_STM-easyedapro:10kΩ
- removed R32: 100kΩ, ProPrj_STM-easyedapro:R0603, symbol ProPrj_STM-easyedapro:100kΩ
- removed SPI1: SPI, ProPrj_STM-easyedapro:JST-XH-06-PACKAGE-LONG-PAD, symbol ProPrj_STM-easyedapro:SPI
- removed USB1: TYPE-C 16PIN 2MD(073), ProPrj_STM-easyedapro:USB-C-SMD_TYPE-C-6PIN-2MD-073, symbol ProPrj_STM-easyedapro:TYPE-C 16PIN 2MD(073)
- removed VIN1: XT60PW-F, ProPrj_STM-easyedapro:CONN-TH_XT60PW-M, symbol ProPrj_STM-easyedapro:XT60PW-F
- removed VOUT1: XT60PW-M, ProPrj_STM-easyedapro:CONN-TH_XT60PW-M, symbol ProPrj_STM-easyedapro:XT60PW-M
- added BOOT1, RESET1: Tactile Button, 160gf, PCM_JLCPCB:SW_TS-1088-AR02016, symbol JLCPCB-Connectors_Buttons:Tactile Button, 160gf, 12V, 50mA, 4.0mm
- added C30: 1uF, PCM_JLCPCB:C_0402, symbol JLCPCB-Capacitors:0402,1uF
- added C31: 100nF, PCM_JLCPCB:C_0402, symbol JLCPCB-Capacitors:0402,100nF
- added GPIO1, SPI/I2C1: 2541WV-08P, easyeda2kicad:HDR-TH_8P-P2.54-V-M-4, symbol easyeda2kicad:2541WV-08P
- added R22, R23, R25, R26: 10kΩ, PCM_JLCPCB:R_0402, symbol JLCPCB-Resistors:0402,10kΩ
- added R27, R28: 47Ω, PCM_JLCPCB:R_0402, symbol JLCPCB-Resistors:0402,47Ω
- added R29: 100kΩ, PCM_JLCPCB:R_0402, symbol JLCPCB-Resistors:0402,100kΩ
- added USB1: TYPE-C 16PIN 2MD, easyeda2kicad:USB-C-SMD_TYPE-C-16PIN-2MD-073, symbol easyeda2kicad:TYPE-C16PIN2MD
- added VIN1, VOUT1: XT60PW-M, easyeda2kicad:CONN-TH_XT60PW-M, symbol easyeda2kicad:XT60PW-M
- C29: renamed from C24; footprint ProPrj_STM-easyedapro:C0402 -> Capacitor_SMD:C_0402_1005Metric
- R19: renamed from R26; footprint ProPrj_STM-easyedapro:R0402 -> Resistor_SMD:R_0402_1005Metric
- R20: renamed from R27; footprint ProPrj_STM-easyedapro:R0402 -> Resistor_SMD:R_0402_1005Metric
- R21: renamed from R28; footprint ProPrj_STM-easyedapro:R0402 -> Resistor_SMD:R_0402_1005Metric
- R24: renamed from R29; footprint ProPrj_STM-easyedapro:R0402 -> Resistor_SMD:R_0402_1005Metric
Connections:
- net 3V3: now also BOOT1.2 (B), GPIO1.2, R23.1, R25.1, SPI/I2C1.2; no longer ST-LINK1.4
- net BOOT0: now also BOOT1.1 (A), R22.1
- net CS: now also SPI/I2C1.6
- net GND: now also C30.2, C31.2, GPIO1.1, R22.2, R26.2, R29.2, RESET1.1 (A), SPI/I2C1.1, USB1.A1B12 (GND), USB1.B1A12 (GND), VIN1.1 (-), VIN1.3, VIN1.4, VOUT1.1 (-), VOUT1.3, VOUT1.4
- net MISO: now also SPI/I2C1.4
- net MOSI: now also SPI/I2C1.3
- net NTC100K: now also C31.1, R29.1
- net PB12: now also GPIO1.3
- net PB13: now also GPIO1.4
- net PB14: now also GPIO1.5
- net PB15: now also GPIO1.6
- net PC6: now also GPIO1.7
- net PC7: now also GPIO1.8
- net SCK: now also SPI/I2C1.5
- net SCL: now also SPI/I2C1.8
- net SDA: now also SPI/I2C1.7
- net SWCLK: now also R26.1, R28.1; no longer ST-LINK1.3
- net SWDIO: now also R25.2, R27.1; no longer ST-LINK1.2
- net USB_DM: now also USB1.A7 (Dn1), USB1.B7 (Dn2)
- net USB_DP: now also USB1.A6 (Dp1), USB1.B6 (Dp2)
- net VIN: now also VIN1.2 (+)
- net VOUT: now also VOUT1.2 (+)
- net at R21.1: now also USB1.A5 (CC1)
- net at R24.1: now also USB1.B5 (CC2)
- net at C29.2, R19.2: now also USB1.A4B9 (VBUS), USB1.B4A9 (VBUS)
- new net: C30.1, R23.2
- new net: R28.2, ST-LINK1.2
- new net: R27.2, ST-LINK1.3
- new net NRST: RESET1.2 (B), ST-LINK1.4
Other:
- note added: "reset switch"
- moved on the sheet: NTC100K1, UART1

Commit message: changes
Parts:
- removed FAN1: HDR-F-2.54_1x4, ProPrj_STM-easyedapro:HDR-F-2.54_1X4, symbol ProPrj_STM-easyedapro:HDR-F-2.54_1x4
- removed NTC100K1: HDR-F-2.54_1x2, ProPrj_STM-easyedapro:HDR-F-2.54_1X2, symbol ProPrj_STM-easyedapro:HDR-F-2.54_1x2
- removed ST-LINK1: ST-Link, ProPrj_STM-easyedapro:JST-XH-04-PACKAGE-LONG-PAD, symbol ProPrj_STM-easyedapro:ST-Link
- removed UART1: UART, ProPrj_STM-easyedapro:JST-XH-04-PACKAGE-LONG-PAD, symbol ProPrj_STM-easyedapro:UART
- added H1: TEMP, easyeda2kicad:HDR-TH_2P-P2.54-V-M, symbol easyeda2kicad:PZ254V-11-02P
- added H2: PZ254V-11-04P_C2691448, easyeda2kicad:HDR-TH_4P-P2.54-V-M, symbol easyeda2kicad:PZ254V-11-04P_C2691448
- added ST_LINK1, UART1: B4B-XH-A, easyeda2kicad:CONN-TH_B4B-XH-A-LF-SN, symbol easyeda2kicad:B4B-XH-A
Connections:
- net +10V: now also H2.2
- net 3V3: now also H1.1, UART1.4
- net FAN: now also H2.4
- net GND: now also H2.1, ST_LINK1.1, UART1.1
- net NRST: now also ST_LINK1.4
- net NTC100K: now also H1.2
- net RX: now also UART1.3
- net TX: now also UART1.2
- net at R28.2: now also ST_LINK1.2
- net at R27.2: now also ST_LINK1.3

Commit message: started layout
Parts:
- added D10, D11: 85V, PCM_JLCPCB:D_SMC, symbol JLCPCB-Diodes:TVS-Uni,5.0SMDJ85CA
Connections:
- net GND: now also D10.2, D11.2
- net NRST: now also C30.1, R23.2
- net VIN: now also D10.1
- net VOUT: now also D11.1
Other:
- moved on the sheet: C30
