File: hardware/KiCad/ProPrj_STM32 MPPT_2024-07-25_15-40-35_2026-05-30.kicad_pcb (KiCad board)
At the start: 2 copper layers, 80 x 100 mm, 117 parts

Commit message: changes
Signed-off-by: DefinitlyNotAHackerTrustMeIAmADolphin <metalhead.baschi@live.de>
Parts:
- removed C37, C39: , ProPrj_STM-easyedapro:C0402
- removed C38: , ProPrj_STM-easyedapro:CAP-SMD_BD6.3-L6.6-W6.6-FD
- removed C40: , ProPrj_STM-easyedapro:C0603
- removed C41, C42, C43, C44, C45, C46, C48, C49, C50, C51, C52, C53: , ProPrj_STM-easyedapro:CAP-TH_BD10.0-P5.00-D1.0-FD
- removed FAN: , ProPrj_STM-easyedapro:HDR-F-2.54_1X4
- removed I2C, ST-LINK1: , ProPrj_STM-easyedapro:JST-XH-04-PACKAGE-LONG-PAD
- removed NTC100K: , ProPrj_STM-easyedapro:HDR-F-2.54_1X2
- removed Q5, Q6, Q7, Q8: , ProPrj_STM-easyedapro:TO-220-3_L10.0-W4.5-P2.54-L
- removed R37, R38, R41, R42, R45, R46: , ProPrj_STM-easyedapro:R0603
- removed RESET: , ProPrj_STM-easyedapro:SW-SMD_4P-L5.1-W5.1-P3.70-LS6.5-TL-2
- removed SPI1: , ProPrj_STM-easyedapro:JST-XH-06-PACKAGE-LONG-PAD
- removed U8, U9: , ProPrj_STM-easyedapro:SOIC-8_L4.9-W3.9-P1.27-LS6.0-BL-EP3.1-1
- removed UA, UB: , ProPrj_STM-easyedapro:SOIC-8_L5.0-W4.0-P1.27-LS6.0-BL
- added C15: 330uF, easyeda2kicad:CAP-TH_BD12.5-P5.00-D0.6-FD, F.Cu at (26.4, 27.9)
- added C17: 330uF, easyeda2kicad:CAP-TH_BD12.5-P5.00-D0.6-FD, F.Cu at (40.1, 27.9)
- added C18: 330uF, easyeda2kicad:CAP-TH_BD12.5-P5.00-D0.6-FD, F.Cu at (40.1, 41.6)
- added C19: 10uF, PCM_JLCPCB:C_0603, F.Cu at (69.1, 62.2)
- added C25: 470nF, PCM_JLCPCB:C_0603, F.Cu at (69.1, 64.5)
- added C28: 100nF, PCM_JLCPCB:C_0402, F.Cu at (47.2, 79.7)
- added C29: 1uF, Capacitor_SMD:C_0402_1005Metric, F.Cu at (56.9, 100.5)
- added CC_Boot1: 100nF, PCM_JLCPCB:C_0603, F.Cu at (70.6, 104.4)
- added C_IN1: 2.2uF, easyeda2kicad:C1210, F.Cu at (65.6, 94.2)
- added C_IN2: 2.2uF, easyeda2kicad:C1210, F.Cu at (65.6, 98.5)
- added C_IN_BYPASS1: 100nF, PCM_JLCPCB:C_0805, F.Cu at (78.4, 93.5)
- added C_OUT1: 22uF, PCM_JLCPCB:C_0805, F.Cu at (78.4, 96.6)
- added C_OUT2: 22uF, PCM_JLCPCB:C_0805, F.Cu at (78.4, 99.6)
- added D7: SS510, PCM_JLCPCB:D_SMA, F.Cu at (80.3, 103.4)
- added H1: TEMP, easyeda2kicad:HDR-TH_2P-P2.54-V-M, F.Cu at (56.3, 107.6)
- added H2: PZ254V-11-04P_C2691448, easyeda2kicad:HDR-TH_4P-P2.54-V-M, F.Cu at (47.4, 107.6)
- added Q1: BSC030N08NS5, easyeda2kicad:TDSON-8_L5.9-W5.2-P1.27-BL-1, F.Cu at (46.4, 53.5)
- added Q2: BSC030N08NS5, easyeda2kicad:TDSON-8_L5.9-W5.2-P1.27-BL-1, F.Cu at (53.0, 53.5)
- added Q3: BSC030N08NS5, easyeda2kicad:TDSON-8_L5.9-W5.2-P1.27-BL-1, F.Cu at (59.6, 53.5)
- added Q4: BSC030N08NS5, easyeda2kicad:TDSON-8_L5.9-W5.2-P1.27-BL-1, F.Cu at (66.2, 53.5)
- added R33: 15kΩ, PCM_JLCPCB:R_0603, F.Cu at (74.4, 99.9)
- added R34: 430kΩ, PCM_JLCPCB:R_0603, F.Cu at (74.4, 102.1)
- added R35: 47kΩ, PCM_JLCPCB:R_0603, F.Cu at (74.4, 104.4)
- added R7: 5.1Ω, PCM_JLCPCB:R_0603, F.Cu at (58.0, 62.2)
- added R8: 5.1Ω, PCM_JLCPCB:R_0603, F.Cu at (58.0, 64.5)
- added RESET1: Tactile Button, 160gf, PCM_JLCPCB:SW_TS-1088-AR02016, F.Cu at (56.1, 116.2)
- added SPI/I2C1: 2541WV-08P, easyeda2kicad:HDR-TH_8P-P2.54-V-M-4, F.Cu at (49.7, 89.6)
- added ST_LINK1: B4B-XH-A, easyeda2kicad:CONN-TH_B4B-XH-A-LF-SN, F.Cu at (48.6, 95.6)
- added UA1: IRS21867STRPBF, JLCPCB:SOIC-8_L5.0-W4.0-P1.27-LS6.0-BL, F.Cu at (46.1, 69.0)
- added UB1: IRS21867STRPBF, JLCPCB:SOIC-8_L5.0-W4.0-P1.27-LS6.0-BL, F.Cu at (52.2, 69.0)
- BOOT1: value (none) -> Tactile Button, 160gf; footprint ProPrj_STM-easyedapro:HDR-F-2.54_1X3 -> PCM_JLCPCB:SW_TS-1088-AR02016
- C1, C2, C3: value (none) -> 100nF; footprint ProPrj_STM-easyedapro:C0603 -> PCM_JLCPCB:C_0402
- C10, C11: value (none) -> 1nF; footprint ProPrj_STM-easyedapro:C0603 -> PCM_JLCPCB:C_0402
- C12: value (none) -> 100nF; footprint ProPrj_STM-easyedapro:C0805 -> PCM_JLCPCB:C_0402
- C13: value (none) -> 10nF; footprint ProPrj_STM-easyedapro:C0805 -> PCM_JLCPCB:C_0402
- C14: value (none) -> 470nF; footprint ProPrj_STM-easyedapro:C0402 -> PCM_JLCPCB:C_0603
- C16, C20, C21, C22, C23: value (none) -> 330uF; footprint ProPrj_STM-easyedapro:C0603 -> easyeda2kicad:CAP-TH_BD12.5-P5.00-D0.6-FD
- C24, C7: value (none) -> 10nF; footprint ProPrj_STM-easyedapro:C0603 -> PCM_JLCPCB:C_0402
- C26, C27: value (none) -> 1nF; footprint ProPrj_STM-easyedapro:C0402 -> PCM_JLCPCB:C_0402
- C30: value (none) -> 1uF; footprint ProPrj_STM-easyedapro:C0402 -> PCM_JLCPCB:C_0402
- C31: value (none) -> 100nF; footprint ProPrj_STM-easyedapro:C0402 -> PCM_JLCPCB:C_0402
- C32: value (none) -> 150pF; footprint ProPrj_STM-easyedapro:C0402 -> PCM_JLCPCB:C_0603
- C33: value (none) -> 47pF; footprint ProPrj_STM-easyedapro:C0402 -> PCM_JLCPCB:C_0603
- C34: value (none) -> 100nF; footprint ProPrj_STM-easyedapro:C0402 -> PCM_JLCPCB:C_0603
- C35: value (none) -> 4.7uF; footprint ProPrj_STM-easyedapro:C0402 -> PCM_JLCPCB:C_0603
- C36: value (none) -> 22uF; footprint ProPrj_STM-easyedapro:C0402 -> PCM_JLCPCB:C_0603
- C4: value (none) -> 4.7uF; footprint ProPrj_STM-easyedapro:C0603 -> PCM_JLCPCB:C_0402
- C5: value (none) -> 100nF; footprint ProPrj_STM-easyedapro:C1206 -> PCM_JLCPCB:C_0402
- C6: value (none) -> 4.7uF; footprint ProPrj_STM-easyedapro:CASE-B_3528 -> PCM_JLCPCB:C_0402
- C8: value (none) -> 1uF; footprint ProPrj_STM-easyedapro:C0603 -> PCM_JLCPCB:C_0402
- C9: value (none) -> 10uF; footprint ProPrj_STM-easyedapro:CAP-SMD_BD6.3-L6.6-W6.6-FD -> PCM_JLCPCB:C_0603
- D1, D4: value (none) -> US1M; footprint ProPrj_STM-easyedapro:SMA_L4.3-W2.6-LS5.2-RD -> PCM_JLCPCB:D_SMA
- D2, D3, D5, D6: value (none) -> 1N4148W; footprint ProPrj_STM-easyedapro:SMA_L4.3-W2.6-LS5.2-RD -> PCM_JLCPCB:D_SOD-123
- GPIO1: value (none) -> 2541WV-08P; footprint ProPrj_STM-easyedapro:HDR-F-2.54_1X8 -> easyeda2kicad:HDR-TH_8P-P2.54-V-M-4
- L1: value (none) -> 47uH; footprint ProPrj_STM-easyedapro:INDUCTOR1 -> easyeda2kicad:IND-TH_L32.2-W22.2_CPEX3222L
- L2: value (none) -> 47uH; footprint ProPrj_STM-easyedapro:IND-SMD_L6.0-W6.0 -> easyeda2kicad:IND-SMD_L7.7-W6.6_APS07A30M220
- L3: value (none) -> 4.7uH; footprint ProPrj_STM-easyedapro:IND-SMD_L6.0-W6.0 -> easyeda2kicad:IND-SMD_L2.0-W1.6-B
- LED1: value (none) -> 19-213/Y2C-CQ2R2L/3T(CY); footprint ProPrj_STM-easyedapro:LED0603-RD-YELLOW -> LED_SMD:LED_0603_1608Metric
- LED2: value (none) -> KT-0603R; footprint ProPrj_STM-easyedapro:LED0603-RD -> LED_SMD:LED_0603_1608Metric
- R1, R2: value (none) -> 510Ω; footprint ProPrj_STM-easyedapro:R0603 -> PCM_JLCPCB:R_0402
- R10, R17, R9: value (none) -> 100kΩ; footprint ProPrj_STM-easyedapro:R0603 -> PCM_JLCPCB:R_0603
- R11, R12, R3, R4: value (none) -> 10kΩ; footprint ProPrj_STM-easyedapro:R0603 -> PCM_JLCPCB:R_0402
- R13, R5: value (none) -> 200kΩ; footprint ProPrj_STM-easyedapro:R0603 -> PCM_JLCPCB:R_0603
- R14, R6: value (none) -> 4.7kΩ; footprint ProPrj_STM-easyedapro:R0603 -> PCM_JLCPCB:R_0603
- R15, R16: value (none) -> 5.1Ω; footprint ProPrj_STM-easyedapro:R0603 -> PCM_JLCPCB:R_0603
- R18: value (none) -> 100kΩ; footprint ProPrj_STM-easyedapro:WIRE-SHUNT -> PCM_JLCPCB:R_0603
- R19: value (none) -> 10kΩ; footprint ProPrj_STM-easyedapro:WIRE-SHUNT -> Resistor_SMD:R_0402_1005Metric
- R20: value (none) -> 10kΩ; footprint ProPrj_STM-easyedapro:R0603 -> Resistor_SMD:R_0402_1005Metric
- R21: value (none) -> 5.1kΩ; footprint ProPrj_STM-easyedapro:R0603 -> Resistor_SMD:R_0402_1005Metric
- R22, R23, R25: value (none) -> 10kΩ; footprint ProPrj_STM-easyedapro:WIRE-SHUNT -> PCM_JLCPCB:R_0402
- R24: value (none) -> 5.1kΩ; footprint ProPrj_STM-easyedapro:WIRE-SHUNT -> Resistor_SMD:R_0402_1005Metric
- R26: value (none) -> 10kΩ; footprint ProPrj_STM-easyedapro:R0402 -> PCM_JLCPCB:R_0402
- R27: value (none) -> 47Ω; footprint ProPrj_STM-easyedapro:R0603 -> PCM_JLCPCB:R_0402
- R28: value (none) -> 47Ω; footprint ProPrj_STM-easyedapro:R0402 -> PCM_JLCPCB:R_0402
- R29: value (none) -> 100kΩ; footprint ProPrj_STM-easyedapro:R0402 -> PCM_JLCPCB:R_0402
- R30: value (none) -> 110kΩ; footprint ProPrj_STM-easyedapro:R0402 -> PCM_JLCPCB:R_0603
- R31: value (none) -> 15kΩ; footprint ProPrj_STM-easyedapro:R0603 -> PCM_JLCPCB:R_0603
- R32: value (none) -> 68kΩ; footprint ProPrj_STM-easyedapro:R0603 -> PCM_JLCPCB:R_0603
- U1: value (none) -> STM32F072RBT6; footprint ProPrj_STM-easyedapro:LQFP-64_L10.0-W10.0-P0.50-LS12.0-BL -> easyeda2kicad:LQFP-64_L10.0-W10.0-P0.50-LS12.0-BL
- U2, U3: value (none) -> CC6937S8-3FB020; footprint ProPrj_STM-easyedapro:PWRM-TH_B2415S-1W -> easyeda2kicad:SOP-8_L4.9-W3.9-P1.27-LS6.0-BL
- U4: value (none) -> SCT2A25STER; footprint ProPrj_STM-easyedapro:SOIC-8_L4.9-W3.9-P1.27-LS6.0-BL -> easyeda2kicad:ESOP-8_L4.9-W3.9-P1.27-LS6.0-BL-EP
- U5: value (none) -> SY8120B1ABC; footprint ProPrj_STM-easyedapro:SOIC-8_L4.9-W3.9-P1.27-LS6.0-BL -> easyeda2kicad:SOT-23-6_L2.9-W1.6-P0.95-LS2.8-BL
- UART1: value (none) -> B4B-XH-A; footprint ProPrj_STM-easyedapro:JST-XH-04-PACKAGE-LONG-PAD -> easyeda2kicad:CONN-TH_B4B-XH-A-LF-SN
- USB1: value (none) -> TYPE-C 16PIN 2MD; footprint ProPrj_STM-easyedapro:USB-C-SMD_TYPE-C-6PIN-2MD-073 -> easyeda2kicad:USB-C-SMD_TYPE-C-16PIN-2MD-073
- VIN1, VOUT1: value (none) -> XT60PW-M; footprint ProPrj_STM-easyedapro:CONN-TH_XT60PW-M -> easyeda2kicad:CONN-TH_XT60PW-M
- moved R22 150.3 mm to (40.3, 96.2), turned to 0 degrees
- moved VOUT1 149.6 mm to (33.3, 109.1), turned to 0 degrees
- moved R23 147.3 mm to (40.3, 98.0), turned to 0 degrees
- moved C10 144.4 mm to (44.4, 74.1), turned to 0 degrees
- moved R25 144.3 mm to (40.3, 99.9), turned to 0 degrees
- moved C4 143.8 mm to (91.8, 27.5)
- moved C16 143.1 mm to (26.4, 41.6), turned to 0 degrees
- moved R4 137.2 mm to (50.1, 76.0), turned to 0 degrees
- moved R3 136.8 mm to (50.1, 74.1), turned to 0 degrees
- moved R27 128.0 mm to (40.3, 103.6), turned to 0 degrees
- moved C31 123.7 mm to (40.3, 94.3), turned to 0 degrees
- moved C27 122.4 mm to (47.2, 77.8), turned to 0 degrees
- moved GPIO1 122.2 mm to (49.7, 85.8), turned to 0 degrees
- moved R26 120.5 mm to (40.3, 101.7), turned to 0 degrees
- moved C14 119.6 mm to (69.1, 60.0), turned to 0 degrees
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Connections:
- BOOT1 pad 1: GND -> BOOT0
- BOOT1 pad 2: BOOT0 -> VBAT
- C1 pad 1: GND -> VBAT
- C1 pad 2: 12V -> VSS
- C10 pad 1: GND -> Net-(U2-VREF)
- C10 pad 2: ISENSEOUT -> VSS
- C11 pad 1: GND -> ISENSEIN
- C11 pad 2: ISENSEIN -> VSS
- C12 pad 1: GND -> VBAT
- C12 pad 2: SHUNT_IN+ -> VSS
- C13 pad 1: GND -> VSENSEIN
- C13 pad 2: SHUNT_IN+ -> VSS
- C14 pad 1: GND -> Net-(UA1-VB)
- C14 pad 2: R29_2 -> VS_A
- C16 pad 1: GND -> SHUNT_IN+
- C16 pad 2: 12V -> VSS
- C2 pad 1: VS_B -> VBAT
- C2 pad 2: C2_2 -> VSS
- C20 pad 1: VS_A -> SHUNT_OUT-
- C20 pad 2: U2_4 -> VSS
- C21 pad 1: 12V -> SHUNT_OUT-
- C21 pad 2: GND -> VSS
- C22 pad 1: VS_A -> SHUNT_OUT-
- C22 pad 2: U2_4 -> VSS
- C23 pad 1: VS_B -> SHUNT_OUT-
- C23 pad 2: C2_2 -> VSS
- C24 pad 1: 12V -> VSENSEOUT
- C24 pad 2: GND -> VSS
- C26 pad 1: GND -> Net-(U3-VREF)
- C26 pad 2: VSENSEIN -> VSS
- C27 pad 1: GND -> ISENSEOUT
- C27 pad 2: VSENSEOUT -> VSS
- C3 pad 1: GND -> VBAT
- C3 pad 2: 3V3 -> VSS
- C30 pad 1: GND -> Net-(C30-Pad1)
- C30 pad 2: 3V3 -> VSS
- C31 pad 1: GND -> NTC100K
- C31 pad 2: 3V3 -> VSS
- C32 pad 1: GND -> +10V
- C32 pad 2: 3V3 -> Net-(U4-FB)
- C33 pad 1: GND -> VBAT
- C33 pad 2: 3V3 -> Net-(U5-FB)
- C34 pad 1: GND -> Net-(U5-BS)
- C34 pad 2: 3V3 -> Net-(U5-LX)
- C35 pad 1: GND -> +10V
- C35 pad 2: 3V3 -> VSS
- C36 pad 1: GND -> VBAT
- C36 pad 2: 3V3 -> VSS
- C4 pad 1: GND -> VBAT
- C4 pad 2: 3V3 -> VSS
- C5 pad 1: GND -> VBAT
- C5 pad 2: 3V3 -> VSS
- C6 pad 1: 3V3 -> VBAT
- C6 pad 2: GND -> VSS
- C7 pad 1: U8_3 -> VBAT
- C7 pad 2: 3V3 -> VSS
- C8 pad 1: C8_1 -> VBAT
- C8 pad 2: 12V -> VSS
- C9 pad 1: 12V -> +10V
- C9 pad 2: GND -> VSS
- D1 pad 1: D1_1 -> Net-(UA1-VB)
- D1 pad 2: HO_A -> +10V
- D2 pad 1: D2_1 -> Net-(UA1-HO)
- D2 pad 2: LO_A -> HO_A
- D3 pad 1: D3_1 -> Net-(UA1-LO)
- D3 pad 2: LO_B -> LO_A
- D4 pad 1: D4_1 -> Net-(UB1-VB)
- D4 pad 2: HO_B -> +10V
- D5 pad 1: U8_2 -> Net-(UB1-HO)
- D5 pad 2: GND -> HO_B
- D6 pad 1: D6_1 -> Net-(UB1-LO)
- D6 pad 2: GND -> LO_B
- GPIO1 pad 1: GND -> VSS
- GPIO1 pad 2: 3V3 -> VBAT
- L2 pad 1: U8_2 -> Net-(U4-SW)
- L2 pad 2: 3V3 -> +10V
- L3 pad 1: D6_1 -> Net-(U5-LX)
- L3 pad 2: 12V -> VBAT
- LED1 pad 1: GND -> VSS
- LED1 pad 2: R31_2 -> Net-(LED1-A)
- LED2 pad 1: GND -> VSS
- LED2 pad 2: R32_2 -> Net-(LED2-A)
- R1 pad 1: GND -> Net-(LED1-A)
- R1 pad 2: VSENSEIN -> VBAT
- R10 pad 1: GND -> LO_A
- R10 pad 2: TIM1_CH1N -> VSS
- R11 pad 1: D1_1 -> TIM1_CH1
- R11 pad 2: HO_A -> VSS
- R12 pad 1: D2_1 -> TIM1_CH1N
- R12 pad 2: LO_A -> VSS
- R13 pad 1: GND -> SHUNT_OUT-
- R13 pad 2: TIM1_CH2N -> VSENSEOUT
- R14 pad 1: GND -> VSENSEOUT
- R14 pad 2: TIM1_CH2 -> VSS
- R15 pad 1: GND -> Net-(UB1-HO)
- R15 pad 2: LO_B -> HO_B
- R16 pad 1: HO_B -> Net-(UB1-LO)
- R16 pad 2: VS_B -> LO_B
- R17 pad 1: GND -> HO_B
- R17 pad 2: NTC100K -> VS_B
- R18 pad 1: VIN -> LO_B
- R18 pad 2: SHUNT_IN+ -> VSS
- R19 pad 1: VIN -> VBUS
- R19 pad 2: SHUNT_IN+ -> Net-(C29-Pad2)
- R2 pad 1: VSENSEIN -> Net-(LED2-A)
- R2 pad 2: SHUNT_IN+ -> LED
- R20 pad 1: GND -> VSS
- R20 pad 2: C8_1 -> VBUS
- R21 pad 1: C8_1 -> Net-(USB1-CC1)
- R21 pad 2: 12V -> VSS
- R22 pad 1: SHUNT_OUT- -> BOOT0
- R22 pad 2: VOUT -> VSS
- R23 pad 1: SHUNT_OUT- -> VBAT
- R23 pad 2: VOUT -> Net-(C30-Pad1)
- R24 pad 1: VIN -> Net-(USB1-CC2)
- R24 pad 2: SHUNT_IN+ -> VSS
- R25 pad 1: SHUNT_OUT- -> VBAT
- R25 pad 2: VOUT -> SWDIO
- R26 pad 1: R26_1 -> SWCLK
- R26 pad 2: GND -> VSS
- R27 pad 1: GND -> SWDIO
- R27 pad 2: SWCLK -> Net-(R27-Pad2)
- R28 pad 1: R28_1 -> SWCLK
- R28 pad 2: GND -> Net-(R28-Pad2)
- R29 pad 1: VBUS -> NTC100K
- R29 pad 2: R29_2 -> VSS
- R3 pad 1: GND -> TIM1_CH2
- R3 pad 2: VSENSEOUT -> VSS
- R30 pad 1: GND -> +10V
- R30 pad 2: VBUS -> Net-(U4-FB)
- R31 pad 1: 3V3 -> Net-(U4-FB)
- R31 pad 2: R31_2 -> unconnected-(R31-Pad2)
- R32 pad 1: LED -> VBAT
- R32 pad 2: R32_2 -> Net-(U5-FB)
- R4 pad 1: VSENSEOUT -> TIM1_CH2N
- R4 pad 2: SHUNT_OUT- -> VSS
- R5 pad 1: HO_A -> SHUNT_IN+
- R5 pad 2: VS_A -> VSENSEIN
- R6 pad 1: GND -> VSENSEIN
- R6 pad 2: LO_A -> VSS
- R9 pad 1: GND -> HO_A
- R9 pad 2: TIM1_CH1 -> VS_A
- U1 pad 1: 3V3 -> VBAT
- U1 pad 10: U1_10 -> unconnected-(U1-PC2-Pad10)
- U1 pad 11: U1_11 -> unconnected-(U1-PC3-Pad11)
- U1 pad 12: GND -> VSS
- U1 pad 13: 3V3 -> VBAT
- U1 pad 14: U1_14 -> unconnected-(U1-PA0-Pad14)
- U1 pad 18: GND -> VSS
- U1 pad 19: 3V3 -> VBAT
- U1 pad 22: U1_22 -> unconnected-(U1-PA6-Pad22)
- U1 pad 27: U1_27 -> unconnected-(U1-PB1-Pad27)
- U1 pad 28: U1_28 -> unconnected-(U1-PB2-Pad28)
- U1 pad 3: (no net) -> unconnected-(U1-PC14-OSC32_IN-Pad3)
- U1 pad 31: GND -> VSS
- U1 pad 32: 3V3 -> VBAT
- U1 pad 4: (no net) -> unconnected-(U1-PC15-OSC32_OUT-Pad4)
- U1 pad 40: U1_40 -> unconnected-(U1-PC9-Pad40)
- U1 pad 43: U1_43 -> unconnected-(U1-PA10-Pad43)
- U1 pad 47: GND -> VSS
- U1 pad 48: 3V3 -> VBAT
- U1 pad 5: (no net) -> unconnected-(U1-PF0-OSC_IN-Pad5)
- U1 pad 50: U1_50 -> unconnected-(U1-PA15-Pad50)
- U1 pad 52: U1_52 -> unconnected-(U1-PC11-Pad52)
- U1 pad 53: U1_53 -> unconnected-(U1-PC12-Pad53)
- U1 pad 58: U1_58 -> unconnected-(U1-PB6-Pad58)
- U1 pad 59: U1_59 -> unconnected-(U1-PB7-Pad59)
- U1 pad 6: (no net) -> unconnected-(U1-PF1-OSC_OUT-Pad6)
- U1 pad 61: U1_61 -> unconnected-(U1-PB8-Pad61)
- U1 pad 62: U1_62 -> unconnected-(U1-PB9-Pad62)
- U1 pad 63: GND -> VSS
- U1 pad 64: 3V3 -> VBAT
- U1 pad 8: U1_8 -> unconnected-(U1-PC0-Pad8)
- U1 pad 9: U1_9 -> unconnected-(U1-PC1-Pad9)
- U2 pad 1: GND -> SHUNT_IN+
- U2 pad 2: 12V -> SHUNT_IN+
- U2 pad 3: VS_A -> SHUNT_IN-
- U2 pad 4: U2_4 -> SHUNT_IN-
- U3 pad 1: GND -> SHUNT_OUT+
- U3 pad 2: 12V -> SHUNT_OUT+
- U3 pad 3: VS_B -> SHUNT_OUT-
- U3 pad 4: C2_2 -> SHUNT_OUT-
- U4 pad 1: VIN -> Net-(U4-FB)
- U4 pad 2: GND -> unconnected-(U4-NC-Pad2)
- U4 pad 3: 3V3 -> SHUNT_IN+
- U4 pad 4: (no net) -> Net-(U4-BST)
- U4 pad 5: ISENSEIN -> Net-(U4-SW)
- U4 pad 6: 3V3 -> unconnected-(U4-TM-Pad6)
- U4 pad 7: GND -> Net-(U4-EN)
- U4 pad 8: SHUNT_IN+ -> VSS
- U5 pad 1: SHUNT_OUT- -> Net-(U5-BS)
- U5 pad 2: GND -> VSS
- U5 pad 3: 3V3 -> Net-(U5-FB)
- U5 pad 4: (no net) -> +10V
- U5 pad 5: ISENSEOUT -> +10V
- U5 pad 6: 3V3 -> Net-(U5-LX)
- UART1 pad 1: GND -> VSS
- UART1 pad 4: 3V3 -> VBAT
- USB1 pad 13: GND -> unconnected-(USB1-EH-Pad13)
- USB1 pad 14: GND -> unconnected-(USB1-EH-Pad14)
- VIN1 pad 1: GND -> VSS
- VIN1 pad 2: VIN -> SHUNT_IN-
- VIN1 pad 3: GND -> VSS
- VIN1 pad 4: GND -> VSS
- VOUT1 pad 1: GND -> VSS
- VOUT1 pad 2: VOUT -> SHUNT_OUT+
- VOUT1 pad 3: GND -> VSS
- VOUT1 pad 4: GND -> VSS
Routing:
- net GND: track 336.0 -> 0.00 mm, vias 164 -> 0
- net 3V3: track 255.8 -> 0.00 mm, vias 8 -> 0
- net SHUNT_IN+: track 118.9 -> 0.00 mm
- net VS_B: track 106.2 -> 0.00 mm, vias 4 -> 0
- net VS_A: track 104.8 -> 0.00 mm, vias 4 -> 0
- net SHUNT_OUT-: track 93.5 -> 0.00 mm
- net 12V: track 87.3 -> 0.00 mm
- net TIM1_CH2N: track 57.8 -> 0.00 mm, vias 2 -> 0
- net NTC100K: track 54.8 -> 0.00 mm, vias 1 -> 0
- net TIM1_CH1N: track 52.8 -> 0.00 mm, vias 2 -> 0
- net USB_DM: track 50.8 -> 0.00 mm, vias 2 -> 0
- net USB_DP: track 49.3 -> 0.00 mm, vias 2 -> 0
- net VSENSEIN: track 47.4 -> 0.00 mm
- net TIM1_CH2: track 45.5 -> 0.00 mm
- net ISENSEIN: track 44.2 -> 0.00 mm
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- removed copper zone on B.Cu, net GND
- removed copper zone on F.Cu, net GND
- removed copper zone on B.Cu, net SHUNT_IN+
- removed copper zone on B.Cu, net SHUNT_OUT-
- removed copper zone on B.Cu, net VS_A
- removed copper zone on B.Cu, net VS_B
Other:
- board outline removed
- board text removed: "12-80V 20A"
- board text removed: "12V"
- board text removed: "3V3"
- board text removed: "CLK"
- board text removed: "CS"
- board text removed: "DIO"
- board text removed: "GND"
- board text removed: "MISO"
- board text removed: "MOSI"
- board text removed: "NC"
- board text removed: "OpenMPPT 1.0"
- board text removed: "PB12"
- board text removed: "PB13"
- board text removed: "PB14"
- board text removed: "PB15"
- board text removed: "PC6"
- board text removed: "PC7"
- board text removed: "PWM"
- board text removed: "RX"
- board text removed: "SCK"
- board text removed: "SCL"
- board text removed: "SDA"
- board text removed: "TX"

Commit message: started layout
Parts:
- removed C1, C2, C3, C5: 100nF, PCM_JLCPCB:C_0402
- removed C4, C6: 4.7uF, PCM_JLCPCB:C_0402
- removed C7: 10nF, PCM_JLCPCB:C_0402
- removed C8: 1uF, PCM_JLCPCB:C_0402
- added C_VDD1: 100nF, PCM_JLCPCB:C_0402, F.Cu at (149.7, 98.4)
- added C_VDD2: 100nF, PCM_JLCPCB:C_0402, F.Cu at (134.0, 99.7)
- added C_VDD3: 100nF, PCM_JLCPCB:C_0402, F.Cu at (134.0, 105.9)
- added C_VDD4: 4.7uF, PCM_JLCPCB:C_0402, F.Cu at (134.0, 98.7)
- added C_VDDA1: 10nF, PCM_JLCPCB:C_0402, F.Cu at (138.6, 94.4)
- added C_VDDA2: 1uF, PCM_JLCPCB:C_0402, F.Cu at (139.6, 94.4)
- added C_VDDIO1: 100nF, PCM_JLCPCB:C_0402, F.Cu at (145.4, 110.1)
- added C_VDDIO2: 4.7uF, PCM_JLCPCB:C_0402, F.Cu at (146.4, 110.1)
- added D10: 85V, PCM_JLCPCB:D_SMC, F.Cu at (106.7, 111.3)
- added D11: 85V, PCM_JLCPCB:D_SMC, F.Cu at (160.4, 111.0)
- added D8: 12V, PCM_JLCPCB:DFN2020-3_L2.0-W2.0-P0.65-BR-1, F.Cu at (128.3, 84.2)
- added D9: 3.3V, PCM_JLCPCB:D_DFN0603-2L, F.Cu at (132.8, 94.1)
- moved VOUT1 127.5 mm to (160.3, 120.1), turned to 90 degrees
- moved C26 120.8 mm to (164.4, 105.3)
- moved C27 120.1 mm to (164.4, 104.0)
- moved C28 119.5 mm to (164.5, 102.7)
- moved U3 115.2 mm to (159.5, 104.6), turned to -90 degrees
- moved C20 110.3 mm to (160.3, 57.1)
- moved C21 110.0 mm to (160.3, 69.6)
- moved C24 108.9 mm to (155.2, 88.6), turned to 90 degrees
- moved R29 108.5 mm to (147.6, 91.0)
- moved C22 107.6 mm to (160.5, 82.1)
- moved C23 106.9 mm to (160.5, 94.6)
- moved C31 105.3 mm to (145.5, 91.0), turned to 180 degrees
- moved R25 104.9 mm to (144.3, 113.7), turned to 90 degrees
- moved C15 103.9 mm to (106.2, 94.3), turned to 180 degrees
- moved SPI/I2C1 103.7 mm to (152.4, 103.7), turned to -90 degrees
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Connections:
- net SHUNT_IN- renamed VIN
- net VBAT renamed 3V3
- C10 pad 2: VSS -> GND
- C11 pad 2: VSS -> GND
- C12 pad 2: VSS -> GND
- C13 pad 2: VSS -> GND
- C15 pad 1: SHUNT_IN+ -> Net-(C15-+)
- C15 pad 2: VSS -> GND
- C16 pad 1: SHUNT_IN+ -> Net-(C15-+)
- C16 pad 2: VSS -> GND
- C17 pad 1: SHUNT_IN+ -> Net-(C15-+)
- C17 pad 2: VSS -> GND
- C18 pad 1: SHUNT_IN+ -> Net-(C15-+)
- C18 pad 2: VSS -> GND
- C19 pad 2: VSS -> GND
- C20 pad 1: SHUNT_OUT- -> Net-(C20-+)
- C20 pad 2: VSS -> GND
- C21 pad 1: SHUNT_OUT- -> Net-(C20-+)
- C21 pad 2: VSS -> GND
- C22 pad 1: SHUNT_OUT- -> Net-(C20-+)
- C22 pad 2: VSS -> GND
- C23 pad 1: SHUNT_OUT- -> Net-(C20-+)
- C23 pad 2: VSS -> GND
- C24 pad 2: VSS -> GND
- C26 pad 2: VSS -> GND
- C27 pad 2: VSS -> GND
- C28 pad 2: VSS -> GND
- C29 pad 1: VSS -> GND
- C30 pad 1: Net-(C30-Pad1) -> NRST
- C30 pad 2: VSS -> GND
- C31 pad 2: VSS -> GND
- C35 pad 2: VSS -> GND
- C36 pad 2: VSS -> GND
- C9 pad 2: VSS -> GND
- C_IN1 pad 1: VSS -> GND
- C_IN2 pad 1: VSS -> GND
- C_IN_BYPASS1 pad 2: VSS -> GND
- C_OUT1 pad 2: VSS -> GND
- C_OUT2 pad 2: VSS -> GND
- D7 pad 2: VSS -> GND
- GPIO1 pad 1: VSS -> GND
- H2 pad 1: VSS -> GND
- LED1 pad 1: VSS -> GND
- LED2 pad 1: VSS -> GND
- Q1 pad 5: SHUNT_IN+ -> Net-(C15-+)
- Q2 pad 1: VSS -> GND
- Q2 pad 2: VSS -> GND
- Q2 pad 3: VSS -> GND
- Q3 pad 5: VSS -> GND
- Q4 pad 1: SHUNT_OUT- -> Net-(C20-+)
- Q4 pad 2: SHUNT_OUT- -> Net-(C20-+)
- Q4 pad 3: SHUNT_OUT- -> Net-(C20-+)
- R10 pad 2: VSS -> GND
- R11 pad 2: VSS -> GND
- R12 pad 2: VSS -> GND
- R13 pad 1: SHUNT_OUT- -> Net-(C20-+)
- R14 pad 2: VSS -> GND
- R18 pad 2: VSS -> GND
- R20 pad 1: VSS -> GND
- R21 pad 2: VSS -> GND
- R22 pad 2: VSS -> GND
- R23 pad 2: Net-(C30-Pad1) -> NRST
- R24 pad 2: VSS -> GND
- R26 pad 2: VSS -> GND
- R29 pad 2: VSS -> GND
- R3 pad 2: VSS -> GND
- R33 pad 2: VSS -> GND
- R35 pad 2: VSS -> GND
- R4 pad 2: VSS -> GND
- R5 pad 1: SHUNT_IN+ -> Net-(C15-+)
- R6 pad 2: VSS -> GND
- RESET1 pad 1: VSS -> GND
- SPI/I2C1 pad 1: VSS -> GND
- ST_LINK1 pad 1: VSS -> GND
- U1 pad 12: VSS -> GND
- U1 pad 31: VSS -> GND
- U1 pad 47: VSS -> GND
- U1 pad 63: VSS -> GND
- U2 pad 1: SHUNT_IN+ -> Net-(C15-+)
- U2 pad 2: SHUNT_IN+ -> Net-(C15-+)
- U2 pad 5: VSS -> GND
- U3 pad 1: SHUNT_OUT+ -> Net-(C20-+)
- U3 pad 2: SHUNT_OUT+ -> Net-(C20-+)
- U3 pad 3: SHUNT_OUT- -> VOUT
- U3 pad 4: SHUNT_OUT- -> VOUT
- U3 pad 5: VSS -> GND
- U4 pad 8: VSS -> GND
- U4 pad 9: VSS -> GND
- U5 pad 2: VSS -> GND
- UA1 pad 4: VSS -> GND
- UART1 pad 1: VSS -> GND
- UB1 pad 4: VSS -> GND
- USB1 pad A1B12: VSS -> GND
- USB1 pad B1A12: VSS -> GND
- VIN1 pad 1: VSS -> GND
- VIN1 pad 3: VSS -> GND
- VIN1 pad 4: VSS -> GND
- VOUT1 pad 1: VSS -> GND
- VOUT1 pad 2: SHUNT_OUT+ -> VOUT
- VOUT1 pad 3: VSS -> GND
- VOUT1 pad 4: VSS -> GND
