File: hardware/KiCad/mcu.kicad_sch (KiCad schematic)
At the start: 13 parts, among them U1 STM32F072RBT6

Commit message: Vendor easyeda2kicad component library; rename project files; fix stale part data
Vendors the 16 easyeda2kicad:* parts (symbols/footprints/3D models) that
were referenced but never committed, registers them in sym-lib-table and
a new fp-lib-table, and adds the EASYEDA2KICAD project text variable so
existing 3D-model paths resolve.

Also corrects BSC030N08NS5's stale metadata (was pointing at an ElecSuper
clone, C49108769, instead of the genuine Infineon part, C501507) and
swaps its footprint to the freshly-fetched one, and fixes STANDARDS.md's
Hardware Universe table (stale reference designators, stale MOSFET/
CC6937 LCSC numbers, ~13 previously undocumented parts, wrong library
path).

Renames the auto-generated project/sheet filenames to something legible:
ProPrj_STM32 MPPT_2024-07-25_15-40-35_2026-05-30.* -> openMPPT_v1.3.*,
and the numbered "N_Name Stuff.kicad_sch" sheets -> mcu/buck_boost/
connectors.kicad_sch. Verified via kicad-cli ERC/DRC before and after -
same violation counts, no structural breakage.

Co-Authored-By: Claude Sonnet 5 <noreply@anthropic.com>
Claude-Session: https://claude.ai/code/session_01FKwww6crXDCSrRUFRETJEs
Parts:
- removed LED1: 19-213/Y2C-CQ2R2L/3T(CY), LED_SMD:LED_0603_1608Metric, symbol ProPrj_STM-easyedapro:19-213/Y2C-CQ2R2L/3T(CY)
- added LED1: KT-0603R, LED_SMD:LED_0603_1608Metric, symbol ProPrj_STM-easyedapro:KT-0603R
Connections:
- net GND: now also LED1.1 (K)
- net at R1.1: now also LED1.2 (A)
