File: hardware/KiCad/power.kicad_sch (KiCad schematic)
At the start: 24 parts, among them U4 SCT2A25STER, U5 SY8120B1ABC

Commit message: fix(hardware): remove D9 (H3V3L06B) TVS diode from power.kicad_sch
Completes the removal decided in 4070cb0 ("docs: remove D9 (H3V3L06B)
3.3V TVS, verified it cannot do its job") - that commit documented the
decision but the schematic instance itself hadn't been deleted yet.
Removes the D9 symbol instance and its now-orphaned cached library
symbol definition.

Co-Authored-By: Claude Sonnet 5 <noreply@anthropic.com>
Claude-Session: https://claude.ai/code/session_018pci5pMUxpfFa5RN5eKA6b
Parts:
- removed D9: 3.3V, PCM_JLCPCB:D_DFN0603-2L, symbol JLCPCB-Diodes:TVS-Bi,H3V3L06B
Changed lines of the file:
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@@
 	)
 	(junction
-		(at 137.16 142.24)
-		(diameter 0)
-		(color 0 0 0 0)
-	)
-	(junction
 		(at 81.28 128.27)
 		(diameter 0)
@@
 	)
 	(junction
-		(at 127 165.1)
-		(diameter 0)
-		(color 0 0 0 0)
-	)
-	(junction
 		(at 73.66 55.88)
 		(diameter 0)
@@
 	(wire
 		(pts
-			(xy 137.16 142.24) (xy 137.16 149.86)
-		)
-		(stroke
-			(width 0)
-			(type default)
-		)
-	)
-	(wire
-		(pts
 			(xy 127 142.24) (xy 127 149.86)
 		)
@@
 	(wire
 		(pts
-			(xy 127 142.24) (xy 137.16 142.24)
+			(xy 127 142.24) (xy 139.7 142.24)
 		)
 		(stroke
@@
 	(wire
 		(pts
-			(xy 137.16 142.24) (xy 139.7 142.24)
-		)
-		(stroke
-			(width 0)
-			(type default)
-		)
-	)
-	(wire
-		(pts
 			(xy 110.49 157.48) (xy 110.49 165.1)
 		)
@@
 	(wire
 		(pts
-			(xy 137.16 157.48) (xy 137.16 165.1)
-		)
-		(stroke
-			(width 0)
-			(type default)
-		)
-	)
-	(wire
-		(pts
 			(xy 100.33 74.93) (xy 107.95 74.93)
 		)
@@
 	(wire
 		(pts
-			(xy 137.16 165.1) (xy 127 165.1)
-		)
-		(stroke
-			(width 0)
-			(type default)
-		)
-	)
-	(wire
-		(pts
 			(xy 106.68 63.5) (xy 107.95 63.5)
 		)
@@
 					(unit 1)
 				)
-			)
-		)
-	)
-	(symbol
-		(lib_id "JLCPCB-Diodes:TVS-Bi,H3V3L06B")
-		(at 137.16 153.67 0)
-		(unit 1)
-		(body_style 1)
-		(exclude_from_sim no)
-		(in_bom yes)
-		(on_board yes)
-		(in_pos_files yes)
-		(dnp no)
-		(fields_autoplaced yes)
-		(property "Reference" "D9"
-			(at 140.97 152.3999 0)
-			(show_name no)
-			(do_not_autoplace no)
-			(effects
-				(font
-					(size 1.27 1.27)
-				)
-				(justify left)
-			)
-		)
-		(property "Value" "3.3V"
-			(at 140.97 154.94 0)
-			(show_name no)
-			(do_not_autoplace no)
-			(effects
-				(font
-					(size 0.8 0.8)
-				)
-				(justify left)
-			)
-		)
-		(property "Footprint" "PCM_JLCPCB:D_DFN0603-2L"
-			(at 135.382 153.67 90)
-			(hide yes)
-			(show_name no)
-			(do_not_autoplace no)
-			(effects
-				(font
-					(size 1.27 1.27)
-				)
-			)
-		)
-		(property "Datasheet" "https://wmsc.lcsc.com/wmsc/upload/file/pdf/v2/lcsc/2401261524_hongjiacheng-H3V3L06B_C20615778.pdf"
-			(at 137.16 153.67 0)
-			(hide yes)
-			(show_name no)
-			(do_not_autoplace no)
-			(effects
-				(font
-					(size 1.27 1.27)
-				)
-			)
-		)
-		(property "Description" "8A 10V 80W 6V Bidirectional 3.3V DFN0603-2L ESD and Surge Protection (TVS/ESD) ROHS"
-			(at 137.16 153.67 0)
-			(hide yes)
-			(show_name no)
-			(do_not_autoplace no)
-			(effects
-				(font
-					(size 1.27 1.27)
-				)
-			)
-		)
-		(property "LCSC" "C20615778"
-			(at 137.16 153.67 0)
-			(hide yes)
-			(show_name no)
-			(do_not_autoplace no)
-			(effects
-				(font
-					(size 1.27 1.27)
-				)
-			)
-		)
-		(property "Stock" "6297"
-			(at 137.16 153.67 0)
-			(hide yes)
-			(show_name no)
-			(do_not_autoplace no)
-			(effects
-				(font
-					(size 1.27 1.27)
-				)
-			)
-		)
-		(property "Price" "0.014USD"
-			(at 137.16 153.67 0)
-			(hide yes)
-			(show_name no)
-			(do_not_autoplace no)
-			(effects
-				(font
-					(size 1.27 1.27)
-				)
-			)
-		)
-		(property "Process" "SMT"
-			(at 137.16 153.67 0)
-			(hide yes)
-			(show_name no)
-			(do_not_autoplace no)
-			(effects
-				(font
-					(size 1.27 1.27)
-				)
-			)
-		)
-		(property "Minimum Qty" "20"
-			(at 137.16 153.67 0)
-			(hide yes)
-			(show_name no)
-			(do_not_autoplace no)
-			(effects
-				(font
-					(size 1.27 1.27)
-				)
-			)
-		)
-		(property "Attrition Qty" "12"
-			(at 137.16 153.67 0)
-			(hide yes)
-			(show_name no)
-			(do_not_autoplace no)
-			(effects
-				(font
-					(size 1.27 1.27)
-				)
-			)
-		)
-		(property "Class" "Preferred Component"
-			(at 137.16 153.67 0)
-			(hide yes)
-			(show_name no)
-			(do_not_autoplace no)
-			(effects
-				(font
-					(size 1.27 1.27)
-				)
-			)
-		)
-		(property "Category" "TVS/Fuse/Board Level Protection,Electrostatic And Surge Protection (TVS/ESD)"
-			(at 137.16 153.67 0)
-			(hide yes)
-			(show_name no)
-			(do_not_autoplace no)
-			(effects
-				(font
-					(size 1.27 1.27)
-				)
-			)
-		)
-		(property "Manufacturer" "hongjiacheng"
-			(at 137.16 153.67 0)
-			(hide yes)
-			(show_name no)
-			(do_not_autoplace no)
-			(effects
-				(font
-					(size 1.27 1.27)
-				)
-			)
-		)
-		(property "Part" "H3V3L06B"
-			(at 137.16 153.67 0)
-			(hide yes)
-			(show_name no)
-			(do_not_autoplace no)
-			(effects
-				(font
-					(size 1.27 1.27)
-				)
-			)
-		)
-		(pin "1"
-		)
-		(pin "2"
-		)
-		(instances
-			(project "openMPPT_v1.3"
-				(path "/b4d74b55-d9ad-45d1-9f37-bb84a2194cf7/ca1cc5b5-a4dc-4cd9-9266-bf9eee57361d"
-					(reference "D9")
-					(unit 1)
-				)
