File: hardware/KiCad/openMPPT_v1.3.kicad_pcb (KiCad board)
At the start: 2 copper layers, 137 parts, among them Q1 BSC030N08NS5, Q2 BSC030N08NS5, Q3 BSC030N08NS5, Q4 BSC030N08NS5, U1 STM32F072RBT6, U2 CC6937S8-3FB020, U3 CC6937S8-3FB020, U4 SCT2A25STER, U5 SY8120B1ABC

Commit message: chore(hardware): sort/reposition PCB components, modernize CONN-TH_B4B-XH-A-LF-SN footprint
Reorganized placement/rotation of ~47 footprints on openMPPT_v1.3.kicad_pcb
ahead of routing. CONN-TH_B4B-XH-A-LF-SN.kicad_mod was re-saved by KiCad 10,
upgrading it from the legacy (module ...) syntax to (footprint ...) like the
earlier HDR-TH_2P-P2.54-V-M cleanup.

Co-Authored-By: Claude Sonnet 5 <noreply@anthropic.com>
Claude-Session: https://claude.ai/code/session_01XCrheiRWP2yQ5mmdKiBeTX
Parts:
- moved C38 117.3 mm to (153.0, 54.0), turned to 180 degrees
- moved C37 115.6 mm to (153.0, 56.0), turned to 180 degrees
- moved C8 114.0 mm to (153.0, 58.0), turned to 180 degrees
- moved C7 112.7 mm to (153.0, 60.0), turned to 180 degrees
- moved C48 112.4 mm to (153.0, 46.0), turned to 180 degrees
- moved C6 111.5 mm to (153.0, 62.0), turned to 180 degrees
- moved C47 110.2 mm to (153.0, 48.0), turned to 180 degrees
- moved C46 108.3 mm to (153.0, 50.0), turned to 180 degrees
- moved C44 108.2 mm to (153.0, 44.0), turned to 180 degrees
- moved C45 106.5 mm to (153.0, 52.0), turned to 180 degrees
- moved D5 94.2 mm to (69.7, 126.4)
- moved Q4 94.2 mm to (69.7, 130.5)
- moved R15 94.2 mm to (73.0, 126.7)
- moved R17 94.2 mm to (73.0, 129.5)
- moved Q3 93.9 mm to (69.5, 139.0)
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