File: hardware/KiCad/connectors.kicad_sch (KiCad schematic)
At the start: 28 parts

Commit message: checked some roadmap things
Parts:
- removed R15: 110kΩ, PCM_JLCPCB:R_0603, symbol JLCPCB-Resistors:0603,110kΩ
