File: hardware/KiCad/buck_boost.kicad_sch (KiCad schematic)
At the start: 73 parts, among them Q1 BSC030N08NS5, Q2 BSC030N08NS5, Q3 BSC030N08NS5, Q4 BSC030N08NS5, U2 CC6937S8-3FB020, U3 CC6937S8-3FB020

Commit message: fix(hardware): add missing Drain pin numbers 6-8 to BSC030N08NS5 schematic symbol
The schematic's cached copy of the BSC030N08NS5 symbol only declared pin
numbers 1-5 (3x Source, Gate, 1x Drain stub), even though the datasheet
(PG-TDSON-8, footnote 1) confirms Drain spans pins 5-8 plus the thermal
pad, all tied together. Pins 6-8 were never added when the symbol's
graphic was redrawn, so Q1-Q4's footprint pads 6/7/8 had no matching
schematic pin and no net ("no pin 6/7/8 in symbol" on netlist update).

Added pins 6-8 stacked at the same coordinate as the existing Drain pin
5 (the standard technique for multi-pin packages where several physical
pins are one net) — schematic renders identically, just with complete
pin-number coverage. Affects all four MOSFETs since they share this
sheet's symbol cache.

Co-Authored-By: Claude Sonnet 5 <noreply@anthropic.com>
Connections:
- net GND: now also Q3.6 (D), Q3.7 (D), Q3.8 (D)
- net IN_CAP: now also Q1.6 (D), Q1.7 (D), Q1.8 (D)
- net VS_A: now also Q2.6 (D), Q2.7 (D), Q2.8 (D)
- net VS_B: now also Q4.6 (D), Q4.7 (D), Q4.8 (D)
